File: Tanque/Control/ControlPCB/ControlPCB.sch (KiCad schematic (older format))
At the start: 7 parts, among them SW1 SW_DPST, SW2 SW_DPST, SW3 SW_DPST, SW4 SW_DPST, U1 nRF24L01+

Commit message: 0.0
Parts:
- added uP1: ARDUPROMINI, symbol ArduProMiniTKB:ARDUPROMINI
Changed lines of the file:
@@
 Wire Wire Line
 	1550 3400 1850 3400
+$Comp
+L ArduProMiniTKB:ARDUPROMINI uP1
+U 1 1 5E708C44
+P 6150 4750
+F 0 "uP1" H 5262 4797 60  0000 C CNN
+F 1 "ARDUPROMINI" H 5262 4691 60  0000 C CNN
+F 2 "" H 6150 4750 60  0000 C CNN
+F 3 "" H 6150 4750 60  0000 C CNN
+	1    6150 4750
+	1    0    0    -1
+$EndComp
 $EndSCHEMATC
